File: distanced/distanced.sch (KiCad schematic (older format))
At the start: 41 parts, among them Y1 Crystal

Commit message: better schematic
Parts:
- removed Y1: Crystal, Crystals:Crystal_SMD_2016-4pin_2.0x1.6mm, symbol Crystal
- added Y1: Crystal_GND24, Crystals:Crystal_SMD_3225-4pin_3.2x2.5mm_HandSoldering, symbol Crystal_GND24
- D3: renamed from D?; footprint (none) -> Diodes_SMD:D_0603
- E1: renamed from E; footprint (none) -> Pin_Headers:Pin_Header_Angled_2x02_Pitch2.54mm
- J1: renamed from J?; footprint (none) -> Pin_Headers:Pin_Header_Angled_1x06_Pitch2.54mm
- J2: renamed from J?; footprint (none) -> Pin_Headers:Pin_Header_Straight_2x03_Pitch2.54mm
- N1: renamed from N; footprint (none) -> Pin_Headers:Pin_Header_Angled_2x02_Pitch2.54mm
- S1: renamed from S; footprint (none) -> Pin_Headers:Pin_Header_Angled_2x02_Pitch2.54mm
- SWRST1: footprint Buttons_Switches_THT:SW_PUSH_6mm_h4.3mm -> Buttons_Switches_SMD:SW_SPST_B3S-1000
- W1: renamed from W; footprint (none) -> Pin_Headers:Pin_Header_Angled_2x02_Pitch2.54mm
- gave numbers to parts that had none: 9
Connections:
- net GNDREF: now also Y1.2, Y1.4
- net at C7.1, uC1.7 ((PCINT6/XTAL1/TOSC1)PB6): now also Y1.1
- net at C8.1, uC1.8 ((PCINT7/XTAL2/TOSC2)PB7): now also Y1.3
