File: distanced/distanced.sch (KiCad schematic (older format))
At the start: 39 parts, among them J1 FTDI prog, J2 ICSP, Q1 BSS138, Q2 BSS138, U1 MIC5205-2.8, Y1 Crystal_GND24

Commit message: Updating the PCB to fit the requirements for PCBway
Parts:
- C1, C3: symbol CP1 -> distanced-rescue:CP1
- C11, C12, C13, C14, C2, C4, C5, C6, C7, C8: symbol C -> distanced-rescue:C
- D1, D2: symbol LED -> distanced-rescue:LED
- D4: symbol D_Small -> distanced-rescue:D_Small
- E1, W1: symbol Conn_02x02_Odd_Even -> distanced-rescue:Conn_02x02_Odd_Even
- J1: symbol Conn_01x06 -> distanced-rescue:Conn_01x06
- J2: symbol Conn_02x03_Odd_Even -> distanced-rescue:Conn_02x03_Odd_Even
- LSR2: symbol VL53L0X -> distanced-rescue:VL53L0X
- Q1, Q2: symbol BSS138 -> distanced-rescue:BSS138
- R1, R10, R11, R12, R13, R2, R3, R4, R5, R8, R9: symbol R -> distanced-rescue:R
- RS485: symbol SP3485CN -> distanced-rescue:SP3485CN
- SWRST1: symbol SW_Push -> distanced-rescue:SW_Push
- U1: symbol MIC5205-2.8 -> distanced-rescue:MIC5205-2.8
- Vreg1: symbol MIC5205-3.3 -> distanced-rescue:MIC5205-3.3
- Y1: symbol Crystal_GND24 -> distanced-rescue:Crystal_GND24
- uC1: symbol ATMEGA328P-AU -> distanced-rescue:ATMEGA328P-AU
Connections:
- net A: now also E1.4 (Pin_4), W1.4 (Pin_4); no longer E1.2 (Pin_2), W1.2 (Pin_2)
- net B: now also E1.2 (Pin_2), W1.2 (Pin_2); no longer E1.4 (Pin_4), W1.4 (Pin_4)

Commit message: Ready for production
Modified silk screen to easy soldering and debugging
Parts:
- C1, C3: symbol distanced-rescue:CP1 -> distanced-rescue:CP1-distanced-rescue
- C11, C12, C13, C14, C2, C4, C5, C6, C7, C8: symbol distanced-rescue:C -> distanced-rescue:C-distanced-rescue
- D1, D2: symbol distanced-rescue:LED -> distanced-rescue:LED-distanced-rescue
- D4: symbol distanced-rescue:D_Small -> distanced-rescue:D_Small-distanced-rescue
- E1, W1: symbol distanced-rescue:Conn_02x02_Odd_Even -> distanced-rescue:Conn_02x02_Odd_Even-distanced-rescue
- J1: symbol distanced-rescue:Conn_01x06 -> distanced-rescue:Conn_01x06-distanced-rescue
- J2: symbol distanced-rescue:Conn_02x03_Odd_Even -> distanced-rescue:Conn_02x03_Odd_Even-distanced-rescue
- LSR2: symbol distanced-rescue:VL53L0X -> distanced-rescue:VL53L0X-distanced-rescue
- Q1, Q2: symbol distanced-rescue:BSS138 -> distanced-rescue:BSS138-distanced-rescue
- R1, R10, R11, R12, R13, R2, R3, R4, R5, R8, R9: symbol distanced-rescue:R -> distanced-rescue:R-distanced-rescue
- RS485: symbol distanced-rescue:SP3485CN -> distanced-rescue:SP3485CN-distanced-rescue
- SWRST1: symbol distanced-rescue:SW_Push -> distanced-rescue:SW_Push-distanced-rescue
- U1: symbol distanced-rescue:MIC5205-2.8 -> distanced-rescue:MIC5205-2.8-distanced-rescue
- Vreg1: symbol distanced-rescue:MIC5205-3.3 -> distanced-rescue:MIC5205-3.3-distanced-rescue
- Y1: symbol distanced-rescue:Crystal_GND24 -> distanced-rescue:Crystal_GND24-distanced-rescue
- uC1: symbol distanced-rescue:ATMEGA328P-AU -> distanced-rescue:ATMEGA328P-AU-distanced-rescue
